Commit message: make zero positions the midpoints

File: URDF/SO100_NEW/so100.urdf (robot description, URDF)
Before this commit: robot so_arm100, 7 links, 6 joints
Joints:
- joint 2: limit lower=0 upper=3.5 effort=35 velocity=1 -> lower=-1.75 upper=1.75 effort=35 velocity=1; origin xyz=0 0.1025 0.0306 rpy=-1.8 0 0 -> xyz=0 0.1025 0.0306 rpy=-0.05 0 0
- joint 3: limit lower=-3.14158 upper=0 effort=35 velocity=1 -> lower=-1.57079 upper=1.57079 effort=35 velocity=1; origin xyz=0 0.11257 0.028 rpy=1.57079 0 0 -> xyz=0 0.11257 0.028 rpy=0 0 0
- joint 4: limit lower=-2.5 upper=1.2 effort=35 velocity=1 -> lower=-1.9764 upper=1.7236 effort=35 velocity=1; origin xyz=0 0.0052 0.1349 rpy=-1 0 0 -> xyz=0 0.0052 0.1349 rpy=-1.5236 0 0
- joint 6: limit lower=-0.2 upper=2.0 effort=35 velocity=1 -> lower=-1.1 upper=1.1 effort=35 velocity=1; origin xyz=-0.0202 -0.0244 0 rpy=0 3.14158 0 -> xyz=-0.0202 -0.0244 0 rpy=0 3.14158 -0.9

Commit message: reverse joint 1 direction

File: URDF/SO100_NEW/so100.urdf (robot description, URDF)
Before this commit: robot so_arm100, 7 links, 6 joints
Joints:
- joint 1: axis 0 1 0 -> 0 -1 0
