Commit message: add back fake joint to top

File: URDF/SO100/so100.urdf (robot description, URDF)
Before this commit: robot so_arm100, 7 links, 6 joints
Links:
- added link Fixed_Jaw_tip
Joints:
- added joint Fixed_Jaw_tip_joint: type fixed, parent gripper, child Fixed_Jaw_tip, origin xyz=0.01 -0.097 0 rpy=0 0 0
- joint 5: origin xyz=0 -0.0601 0 rpy=0 1.57079 0 -> xyz=0 -0.0601 0 rpy=0 3.14158 0
- joint 6: limit lower=-1.1 upper=1.1 effort=35 velocity=1 -> lower=-0.2 upper=2.0 effort=35 velocity=1; origin xyz=-0.0202 -0.0244 0 rpy=0 3.14158 -0.9 -> xyz=-0.0202 -0.0244 0 rpy=0 3.14158 0
