Commit message: first basic version working in meshcat

File: URDF/Piper/piper_description.urdf (robot description, URDF)
Before this commit: robot piper_description, 10 links, 9 joints
Links:
- link base_link: geometry collision mesh filename=/home/alex/git/piper_grip/URDF/Piper/assets/base_link.STL; visual mesh filename=/home/alex/git/piper_grip/URDF/Piper/assets/base_link.STL
- link gripper_base: geometry collision mesh filename=/home/alex/git/piper_grip/URDF/Piper/assets/gripper_base.STL; visual mesh filename=/home/alex/git/piper_grip/URDF/Piper/assets/gripper_base.STL
- link link1: geometry collision mesh filename=/home/alex/git/piper_grip/URDF/Piper/assets/link1.STL; visual mesh filename=/home/alex/git/piper_grip/URDF/Piper/assets/link1.STL
- link link2: geometry collision mesh filename=/home/alex/git/piper_grip/URDF/Piper/assets/link2.STL; visual mesh filename=/home/alex/git/piper_grip/URDF/Piper/assets/link2.STL
- link link3: geometry collision mesh filename=/home/alex/git/piper_grip/URDF/Piper/assets/link3.STL; visual mesh filename=/home/alex/git/piper_grip/URDF/Piper/assets/link3.STL
- link link4: geometry collision mesh filename=/home/alex/git/piper_grip/URDF/Piper/assets/link4.STL; visual mesh filename=/home/alex/git/piper_grip/URDF/Piper/assets/link4.STL
- link link5: geometry collision mesh filename=/home/alex/git/piper_grip/URDF/Piper/assets/link5.STL; visual mesh filename=/home/alex/git/piper_grip/URDF/Piper/assets/link5.STL
- link link6: geometry collision mesh filename=/home/alex/git/piper_grip/URDF/Piper/assets/link6.STL; visual mesh filename=/home/alex/git/piper_grip/URDF/Piper/assets/link6.STL
- link link7: geometry collision mesh filename=/home/alex/git/piper_grip/URDF/Piper/assets/link7.STL; visual mesh filename=/home/alex/git/piper_grip/URDF/Piper/assets/link7.STL
- link link8: geometry collision mesh filename=/home/alex/git/piper_grip/URDF/Piper/assets/link8.STL; visual mesh filename=/home/alex/git/piper_grip/URDF/Piper/assets/link8.STL

Commit message: web server and robot server running

File: URDF/Piper/piper_description.urdf (robot description, URDF)
Before this commit: robot piper_description, 10 links, 9 joints
Links:
- link base_link: geometry collision mesh filename=/home/zhamers/telegrip/URDF/Piper/assets/base_link.STL; visual mesh filename=/home/zhamers/telegrip/URDF/Piper/assets/base_link.STL
- link gripper_base: geometry collision mesh filename=/home/zhamers/telegrip/URDF/Piper/assets/gripper_base.STL; visual mesh filename=/home/zhamers/telegrip/URDF/Piper/assets/gripper_base.STL
- link link1: geometry collision mesh filename=/home/zhamers/telegrip/URDF/Piper/assets/link1.STL; visual mesh filename=/home/zhamers/telegrip/URDF/Piper/assets/link1.STL
- link link2: geometry collision mesh filename=/home/zhamers/telegrip/URDF/Piper/assets/link2.STL; visual mesh filename=/home/zhamers/telegrip/URDF/Piper/assets/link2.STL
- link link3: geometry collision mesh filename=/home/zhamers/telegrip/URDF/Piper/assets/link3.STL; visual mesh filename=/home/zhamers/telegrip/URDF/Piper/assets/link3.STL
- link link4: geometry collision mesh filename=/home/zhamers/telegrip/URDF/Piper/assets/link4.STL; visual mesh filename=/home/zhamers/telegrip/URDF/Piper/assets/link4.STL
- link link5: geometry collision mesh filename=/home/zhamers/telegrip/URDF/Piper/assets/link5.STL; visual mesh filename=/home/zhamers/telegrip/URDF/Piper/assets/link5.STL
- link link6: geometry collision mesh filename=/home/zhamers/telegrip/URDF/Piper/assets/link6.STL; visual mesh filename=/home/zhamers/telegrip/URDF/Piper/assets/link6.STL
- link link7: geometry collision mesh filename=/home/zhamers/telegrip/URDF/Piper/assets/link7.STL; visual mesh filename=/home/zhamers/telegrip/URDF/Piper/assets/link7.STL
- link link8: geometry collision mesh filename=/home/zhamers/telegrip/URDF/Piper/assets/link8.STL; visual mesh filename=/home/zhamers/telegrip/URDF/Piper/assets/link8.STL

Commit message: added stereo implementation but currently white screen

File: URDF/Piper/piper_description.urdf (robot description, URDF)
Before this commit: robot piper_description, 10 links, 9 joints
Links:
- link base_link: geometry collision mesh filename=assets/base_link.STL; visual mesh filename=assets/base_link.STL
- link gripper_base: geometry collision mesh filename=assets/gripper_base.STL; visual mesh filename=assets/gripper_base.STL
- link link1: geometry collision mesh filename=assets/link1.STL; visual mesh filename=assets/link1.STL
- link link2: geometry collision mesh filename=assets/link2.STL; visual mesh filename=assets/link2.STL
- link link3: geometry collision mesh filename=assets/link3.STL; visual mesh filename=assets/link3.STL
- link link4: geometry collision mesh filename=assets/link4.STL; visual mesh filename=assets/link4.STL
- link link5: geometry collision mesh filename=assets/link5.STL; visual mesh filename=assets/link5.STL
- link link6: geometry collision mesh filename=assets/link6.STL; visual mesh filename=assets/link6.STL
- link link7: geometry collision mesh filename=assets/link7.STL; visual mesh filename=assets/link7.STL
- link link8: geometry collision mesh filename=assets/link8.STL; visual mesh filename=assets/link8.STL
