Commit message: change distance between arms, correct left/right arm selection

File: URDF/Piper/dual_piper.urdf (robot description, URDF)
Before this commit: robot piper_description, 20 links, 19 joints
Joints:
- joint base_to_arm2_base_joint: origin xyz=0 -0.5 0.0 rpy=0 0 0 -> xyz=0 -0.57 0.0 rpy=0 0 0

Commit message: adjusted masses and inertias of urdf, added IK with pinocchio, started adding sim interface (this version is not working yet)

File: URDF/Piper/dual_piper.urdf (robot description, URDF)
Before this commit: robot piper_description, 20 links, 19 joints
Links:
- link arm2_base_link: mass 0.333893486740112 -> 1.02
- link arm2_gripper_base: mass 0.145318531013916 -> 0.45
- link arm2_link1: mass 0.215052383265765 -> 0.71
- link arm2_link2: mass 0.463914239236335 -> 1.17
- link arm2_link3: mass 0.219942452993132 -> 0.5
- link arm2_link4: mass 0.131814339939458 -> 0.38
- link arm2_link5: mass 0.134101341225523 -> 0.383
- link arm2_link6: mass 0.00699089613564366 -> 0.007
- link arm2_link7: mass 0.0303534920715906 -> 0.025
- link arm2_link8: mass 0.0303534920715904 -> 0.025
- link base_link: mass 0.333893486740112 -> 1.02
- link gripper_base: mass 0.145318531013916 -> 0.45
- link link1: mass 0.215052383265765 -> 0.71
- link link2: mass 0.463914239236335 -> 1.17
- link link3: mass 0.219942452993132 -> 0.5
- link link4: mass 0.131814339939458 -> 0.38
- link link5: mass 0.134101341225523 -> 0.383
- link link6: mass 0.00699089613564366 -> 0.007
- link link7: mass 0.0303534920715906 -> 0.025
- link link8: mass 0.0303534920715904 -> 0.025
